Commit message: [11]放弃修改rviz显示的问题。使用xacro中重复加载joint_state_publisher插件的方法

File: src/car_model/urdf/smart_v4_解决前轮的显示bug.xacro (robot description, xacro)
@@ -66,5 +66,5 @@
         </inertial>
     </link>
-    <!--Rear Right Wheel-->
+    <!--base_link - rear_right_wheel-->
     <joint name="rear_right_wheel_joint" type="continuous">
         <parent link="base_link"/>
@@ -96,5 +96,5 @@
         </inertial>
     </link>
-    <!--Rear Left Wheel-->
+    <!--base_link - rear_left_wheel-->
     <joint name="rear_left_wheel_joint" type="continuous">
         <parent link="base_link"/>
@@ -126,5 +126,5 @@
         </inertial>
     </link>
-    <!--Front Right Steering-->
+    <!--base_link - front_right_steering - front_right_wheel_link-->
     <joint name="front_right_steering_joint" type="revolute">
         <parent link="base_link"/>
@@ -298,25 +298,4 @@
         </actuator>
     </transmission> -->
-    <!--  -->
-    <transmission name="tran5">
-        <type>transmission_interface/SimpleTransmission</type>
-        <joint name="front_right_wheel_joint">
-            <hardwareInterface>hardware_interface/VelocityJointInterface</hardwareInterface>
-        </joint>
-        <actuator name="motor3">
-            <hardwareInterface>hardware_interface/VelocityJointInterface</hardwareInterface>
-            <mechanicalReduction>1</mechanicalReduction>
-        </actuator>
-    </transmission>
-    <transmission name="tran6">
-        <type>transmission_interface/SimpleTransmission</type>
-        <joint name="front_left_wheel_joint">
-            <hardwareInterface>hardware_interface/VelocityJointInterface</hardwareInterface>
-        </joint>
-        <actuator name="motor4">
-            <hardwareInterface>hardware_interface/VelocityJointInterface</hardwareInterface>
-            <mechanicalReduction>1</mechanicalReduction>
-        </actuator>
-    </transmission>
     <!-- Friction Parametres -->
     <gazebo reference="rear_right_wheel_link">
